File: KiCad/Blaster/Project.kicad_sch (KiCad schematic)
At the start: 0 parts

Commit message: Updated Blaster Microcontroller Schematic
Other:
- sheet Blaster_Bottom renamed Microcontroller
- removed sheet Blaster Top
- added sheet Communications (Communications.kicad_sch)
- sheet Microcontroller: file Blaster_Bottom.kicad_sch -> Microcontroller.kicad_sch
