File: KiCad/Blaster/Blaster_Power.kicad_sch (KiCad schematic)
At the start: 0 parts

Commit message: Blaster Power and Communications schematic updates. Add Revision B schematic
Parts:
- added BT1: 18650, symbol Device:Battery_Cell
- added C1, C2, C4, C5: 4.7µF, symbol Device:C
- added C3, C6, C8: 0.1µF, symbol Device:C
- added C7: 22µF, symbol Device:C
- added D1: Charge, symbol Device:LED_Filled
- added J1: +12V, Connector_AMASS:AMASS_XT60PW-M_1x02_P7.20mm_Horizontal, symbol 0_AKeller_Parts:Header_1x2
- added L1: 6.8µH, symbol Device:L
- added R1, R2: 2.2kΩ, symbol Device:R_US
- added R3: 47kΩ, symbol Device:R_US
- added R4: 15kΩ, symbol Device:R_US
- added SW1: Charge, symbol Switch:SW_SPDT
- added SW2: Power, symbol Switch:SW_SPST
- added TP1: +12V, 0_AKeller_Footprints:1x1_100mil_Header, symbol 0_AKeller_Parts:Test_Point
- added TP2: +5V, 0_AKeller_Footprints:1x1_100mil_Header, symbol 0_AKeller_Parts:Test_Point
- added TP3: Charge, 0_AKeller_Footprints:1x1_100mil_Header, symbol 0_AKeller_Parts:Test_Point
- added TP4: V_{BAT}, 0_AKeller_Footprints:1x1_100mil_Header, symbol 0_AKeller_Parts:Test_Point
- added TP5: Power, 0_AKeller_Footprints:1x1_100mil_Header, symbol 0_AKeller_Parts:Test_Point
- added TP6: +3.3V, 0_AKeller_Footprints:1x1_100mil_Header, symbol 0_AKeller_Parts:Test_Point
- added U1: TLV1117-50, symbol Regulator_Linear:TLV1117-50
- added U2: MCP73831-2-OT, Package_TO_SOT_SMD:SOT-23-5, symbol Battery_Management:MCP73831-2-OT
- added U3: LMR51635, Package_TO_SOT_SMD:SOT-23-6_Handsoldering, symbol 0_AKeller_Parts:LMR51635
Connections:
- new net: R1.2, U2.1 (STAT)
- new net: BT1.1 (+), C4.1, SW2.1 (A), TP4.1, U2.3 (V_{BAT})
- new net: C2.1, D1.2 (A), SW1.2 (B), TP3.1, U2.4 (V_{DD})
- new net: R2.1, U2.5 (PROG)
- new net: R3.2, R4.1, U3.1 (FB)
- new net: D1.1 (K), R1.1
- new net: C5.1, C6.1, SW2.2 (B), TP5.1, U3.2 (EN), U3.3 (VIN)
- new net: C1.1, SW1.1 (A), TP2.1, U1.2 (VO)
- new net: C3.2, L1.1, U3.5 (SW)
- new net: C3.1, U3.6 (CB)
- new net +12V: J1.2, TP1.1, U1.3 (VI)
- new net +3V3: C7.1, C8.1, L1.2, R3.1, TP6.1
- new net GND: BT1.2 (-), C1.2, C2.2, C4.2, C5.2, C6.2, C7.2, C8.2, J1.1, R2.2, R4.2, U1.1 (GND), U2.2 (V_{SS}), U3.4 (GND)
- new net VBUS: SW1.3 (C)
Other:
- note added: "Tether"
- note added: "USB"

Commit message: Assign blaster footprints, Create Blaster PCB Outline
Parts:
- added U4: MCP6002, Package_SO:SOIC-8-1EP_3.9x4.9mm_P1.27mm_EP2.29x3mm, symbol Amplifier_Operational:MCP6002-xMC
- BT1: footprint (none) -> Battery:BatteryHolder_Keystone_1042_1x18650
- C1, C2, C3, C4, C5, C6, C7, C8: footprint (none) -> Capacitor_SMD:C_0805_2012Metric_Pad1.18x1.45mm_HandSolder
- D1: footprint (none) -> LED_SMD:LED_0805_2012Metric_Pad1.15x1.40mm_HandSolder
- L1: footprint (none) -> 0_AKeller_Footprints:LA Blaster Power Inductor
- R1, R2, R3, R4: footprint (none) -> Resistor_SMD:R_0805_2012Metric_Pad1.20x1.40mm_HandSolder
- SW1: footprint (none) -> 0_AKeller_Footprints:SW_SPDT_CK_JS102011SAQN
- U1: footprint (none) -> Package_TO_SOT_SMD:SOT-223-3_TabPin2
- U2: footprint Package_TO_SOT_SMD:SOT-23-5 -> Package_TO_SOT_SMD:SOT-23-5_HandSoldering
Connections:
- net +3V3: now also U4.8 (V+)
- net GND: now also U4.4 (V-), U4.9 (V-)
- no-connect marks 0 -> 3

Commit message: Assign blaster PCB Footprints
Parts:
- SW1: footprint 0_AKeller_Footprints:SW_SPDT_CK_JS102011SAQN -> 0_AKeller_Footprints:T80-T
- SW2: footprint (none) -> 0_AKeller_Footprints:LA Blaster Power Switch
Changed lines of the file:
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@@
 			)
 		)
-		(property "Footprint" ""
+		(property "Footprint" "0_AKeller_Footprints:LA Blaster Power Switch"
 			(at 146.05 95.25 0)
 			(effects
@@
 			)
 		)
-		(property "Footprint" "0_AKeller_Footprints:SW_SPDT_CK_JS102011SAQN"
+		(property "Footprint" "0_AKeller_Footprints:T80-T"
 			(at 91.44 77.47 0)
 			(effects
