File: KiCad/Blaster/Blaster_Power.kicad_sch (KiCad schematic)
At the start: 28 parts, among them J1 +12V, SW1 Charge, SW2 Power, U1 TLV1117-50, U2 MCP73831-2-OT, U3 LMR51635, U4 MCP6002

Commit message: Complete Blaster PCB layout and traces
Parts:
- added D2: Tether, LED_SMD:LED_0805_2012Metric_Pad1.15x1.40mm_HandSolder, symbol Device:LED_Filled
- added D3: Power, LED_SMD:LED_0805_2012Metric_Pad1.15x1.40mm_HandSolder, symbol Device:LED_Filled
- added R2, R5: 1kΩ, Resistor_SMD:R_0805_2012Metric_Pad1.20x1.40mm_HandSolder, symbol Device:R_US
- J1: footprint Connector_AMASS:AMASS_XT60PW-M_1x02_P7.20mm_Horizontal -> 0_AKeller_Footprints:AMASS_XT60PW-M_1x02_P7.20mm_Horizontal
- U4: footprint Package_SO:SOIC-8-1EP_3.9x4.9mm_P1.27mm_EP2.29x3mm -> Package_SO:SOIC-8_3.9x4.9mm_P1.27mm; symbol Amplifier_Operational:MCP6002-xMC -> Amplifier_Operational:MCP6002-xSN
- renumbered C2 to C1, C1 to C2, R2 to R3, R3 to R4, R4 to R6, TP3 to TP1, TP1 to TP2, TP2 to TP3
Connections:
- net +12V: now also D2.2 (A)
- net +3V3: now also D3.2 (A)
- net GND: now also R2.2, R5.2; no longer U4.9 (V-)
- net VBUS: now also SW1.1 (A); no longer SW1.3 (C)
- net at C2.1, TP3.1, U1.2 (VO): now also SW1.3 (C); no longer SW1.1 (A)
- new net: D2.1 (K), R2.1
- new net: D3.1 (K), R5.1
Other:
- moved on the sheet: C2, J1, TP2, TP3, U1
