File: KiCad/Blaster/_autosave-Blaster_Power.kicad_sch (KiCad schematic)
At the start: 28 parts, among them J1 +12V, SW1 Charge, SW2 Power, U1 TLV1117-50, U2 MCP73831-2-OT, U3 LMR51635, U4 MCP6002

Commit message: Place major components on PCB
Parts:
- J1: footprint Connector_AMASS:AMASS_XT60PW-M_1x02_P7.20mm_Horizontal -> 0_AKeller_Footprints:AMASS_XT60PW-M_1x02_P7.20mm_Horizontal
Changed lines of the file:
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@@
 			)
 		)
-		(property "Footprint" "Connector_AMASS:AMASS_XT60PW-M_1x02_P7.20mm_Horizontal"
+		(property "Footprint" "0_AKeller_Footprints:AMASS_XT60PW-M_1x02_P7.20mm_Horizontal"
 			(at 38.1 73.66 0)
 			(effects
