File: KiCad/Blaster/Microcontroller.kicad_sch (KiCad schematic)
At the start: 65 parts, among them J1 ICSP, J11 Solenoid, J2 Speaker, J3 Laser, J4 Laser, Q1 DMG3402L, Q2 DMG3402L, Q3 DMG3402L, Q4 DMG3402L, SW5 Auto, SW6 Burst, SW7 Single, SW8 Trigger, U2 PIC16LF1788, U4 Audio FX Mini, U5 MCP6002

Commit message: Blaster Power and Communications schematic updates. Add Revision B schematic
Parts:
- renumbered C5 to C10, C6 to C11, D4 to D2, D6 to D3, D7 to D4, J1 to J3, J11 to J4, J4 to J5, J3 to J6, Q2 to Q1, Q3 to Q2, Q1 to Q3, R3 to R10, R4 to R11, R13 to R12, R12 to R13, R11 to R14, R10 to R15, R14 to R21, R21 to R22, R9 to R5, R5 to R6, R8 to R7, R6 to R8, R7 to R9, SW8 to SW3, SW7 to SW4, SW6 to SW5, SW5 to SW6, TP1 to TP10, TP1 to TP11, TP3 to TP12, TP5 to TP13, TP4 to TP14, TP6 to TP15, TP1 to TP16, TP7 to TP17, TP2 to TP18, TP11 to TP19, TP12 to TP20, TP16 to TP21, TP13 to TP22, TP14 to TP23, TP15 to TP24, TP18 to TP25, TP19 to TP26, TP20 to TP27, TP21 to TP28, TP17 to TP29, TP22 to TP30, TP23 to TP31, TP8 to TP7, TP9 to TP8, TP10 to TP9, U5 to U4, U4 to U5, U2 to U6

Commit message: Assign blaster footprints, Create Blaster PCB Outline
Parts:
- added R18, R19: 0Ω, Resistor_SMD:R_0805_2012Metric_Pad1.20x1.40mm_HandSolder, symbol Device:R_US
- C9: footprint (none) -> Capacitor_SMD:C_0805_2012Metric_Pad1.18x1.45mm_HandSolder
- D2: footprint 0_AKeller_Footprints:Diode_0805 -> Diode_SMD:D_0805_2012Metric_Pad1.15x1.40mm_HandSolder
- J2, J4, J5, J6: footprint (none) -> 0_AKeller_Footprints:1x2_100mil_Header_Locking
- R10, R11, R12, R13, R14, R15, R16, R17, R5, R6, R7, R8, R9: footprint (none) -> Resistor_SMD:R_0805_2012Metric_Pad1.20x1.40mm_HandSolder
- R20: renamed from R18; footprint (none) -> Resistor_SMD:R_0805_2012Metric_Pad1.20x1.40mm_HandSolder
- R21: renamed from R19; footprint (none) -> Resistor_SMD:R_0805_2012Metric_Pad1.20x1.40mm_HandSolder
- R22: renamed from R20; footprint (none) -> Resistor_SMD:R_0805_2012Metric_Pad1.20x1.40mm_HandSolder
- R23: renamed from R21; footprint (none) -> Resistor_SMD:R_0805_2012Metric_Pad1.20x1.40mm_HandSolder
- R24: renamed from R22; footprint (none) -> Resistor_SMD:R_0805_2012Metric_Pad1.20x1.40mm_HandSolder
- SW3: footprint (none) -> Button_Switch_THT:SW_Tactile_SPST_Angled_PTS645Vx31-2LFS
- SW4, SW5, SW6: footprint (none) -> Button_Switch_THT:SW_PUSH_6mm_H5mm
- U4: footprint Package_DFN_QFN:DFN-8-1EP_3x2mm_P0.5mm_EP1.75x1.45mm -> Package_SO:SOIC-8-1EP_3.9x4.9mm_P1.27mm_EP2.29x3mm
Connections:
- net +3V3: now also R18.1, R19.1; no longer J5.1, J6.1
- new net: J5.1, R18.2
- new net: J6.1, R19.2
Other:
- moved on the sheet: J5, J6

Commit message: Assign blaster PCB Footprints
Parts:
- U5: footprint (none) -> 0_AKeller_Footprints:Adafruit_AudioFXMini
Changed lines of the file:
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@@
 			)
 		)
-		(property "Footprint" ""
+		(property "Footprint" "0_AKeller_Footprints:Adafruit_AudioFXMini"
 			(at 172.72 62.23 0)
 			(effects

Commit message: Complete Blaster PCB layout and traces
Parts:
- removed TP10: MCLR, 0_AKeller_Footprints:1x1_100mil_Header, symbol 0_AKeller_Parts:Test_Point
- removed TP22: Single, 0_AKeller_Footprints:1x1_100mil_Header, symbol 0_AKeller_Parts:Test_Point
- removed TP23: Burst, 0_AKeller_Footprints:1x1_100mil_Header, symbol 0_AKeller_Parts:Test_Point
- removed TP24: Auto, 0_AKeller_Footprints:1x1_100mil_Header, symbol 0_AKeller_Parts:Test_Point
- removed TP25, TP28: Auto LED, 0_AKeller_Footprints:1x1_100mil_Header, symbol 0_AKeller_Parts:Test_Point
- removed TP26, TP30: Burst LED, 0_AKeller_Footprints:1x1_100mil_Header, symbol 0_AKeller_Parts:Test_Point
- removed TP27: Single LED, 0_AKeller_Footprints:1x1_100mil_Header, symbol 0_AKeller_Parts:Test_Point
- removed TP31: Blue PWM, 0_AKeller_Footprints:1x1_100mil_Header, symbol 0_AKeller_Parts:Test_Point
- removed TP8: Ramp, 0_AKeller_Footprints:1x1_100mil_Header, symbol 0_AKeller_Parts:Test_Point
- removed TP9: Audio PWM, 0_AKeller_Footprints:1x1_100mil_Header, symbol 0_AKeller_Parts:Test_Point
- added TP18: Red, 0_AKeller_Footprints:1x1_100mil_Header, symbol 0_AKeller_Parts:Test_Point
- added TP21: Blue, 0_AKeller_Footprints:1x1_100mil_Header, symbol 0_AKeller_Parts:Test_Point
- TP20: value Trigger -> Green
- U4: footprint Package_SO:SOIC-8-1EP_3.9x4.9mm_P1.27mm_EP2.29x3mm -> Package_SO:SOIC-8_3.9x4.9mm_P1.27mm; symbol Amplifier_Operational:MCP6002-xMC -> Amplifier_Operational:MCP6002-xSN
- renumbered D2 to D4, D3 to D5, D4 to D6, R8 to R10, R9 to R11, R10 to R12, R11 to R13, R12 to R14, R13 to R15, R14 to R16, R15 to R17, R16 to R18, R17 to R19, R18 to R20, R19 to R21, R20 to R22, R21 to R23, R22 to R24, R23 to R25, R24 to R26, R5 to R7, R6 to R8, R7 to R9, TP13 to TP10, TP14 to TP11, TP15 to TP12, TP16 to TP13, TP17 to TP14, TP18 to TP15, TP19 to TP16, TP21 to TP17, TP29 to TP19, TP11 to TP8, TP12 to TP9
Connections:
- net +5V is gone; now on net +3V3: J3.2, R12.1
- net Green PWM: now also TP20.1
- net at R14.1, SW3.1, U6.22 (P1C/AN10/RB1): no longer TP20.1
- net at R26.1, U6.12 (RC1/T1OSI/CCP2): now also TP21.1
- net at R23.1, U6.13 (RC2/P1A/CCP1): now also TP18.1
