File: KiCad/Target_Jumper/Target_Jumper.kicad_sch (KiCad schematic)
At the start: 0 parts

Commit message: Target Jumper Schematics
Parts:
- added J1, J10, J11, J12, J13, J14, J15, J16, J17, J18, J2, J3, J4, J5, J6, J7, J8, J9: I2C, symbol 0_AKeller_Parts:Header_1x6
Connections:
- new net: J1.3, J10.3, J11.3, J12.3, J13.3, J14.3, J15.3, J16.3, J17.3, J18.3, J2.3, J3.3, J4.3, J5.3, J6.3, J7.3, J8.3, J9.3
- new net: J1.4, J10.4, J11.4, J12.4, J13.4, J14.4, J15.4, J16.4, J17.4, J18.4, J2.4, J3.4, J4.4, J5.4, J6.4, J7.4, J8.4, J9.4
- new net +5V: J1.1, J1.2, J10.1, J10.2, J11.1, J11.2, J12.1, J12.2, J13.1, J13.2, J14.1, J14.2, J15.1, J15.2, J16.1, J16.2, J17.1, J17.2, J18.1, J18.2, J2.1, J2.2, J3.1, J3.2, J4.1, J4.2, J5.1, J5.2, J6.1, J6.2, J7.1, J7.2, J8.1, J8.2, J9.1, J9.2
- new net GND: J1.5, J1.6, J10.5, J10.6, J11.5, J11.6, J12.5, J12.6, J13.5, J13.6, J14.5, J14.6, J15.5, J15.6, J16.5, J16.6, J17.5, J17.6, J18.5, J18.6, J2.5, J2.6, J3.5, J3.6, J4.5, J4.6, J5.5, J5.6, J6.5, J6.6, J7.5, J7.6, J8.5, J8.6, J9.5, J9.6
Other:
- note added: "1 = +5V 2 = +5V 3 = SCL 4 = SDA 5 = GND 6 = GND"
- company: (none) -> Idaho State University
- title: (none) -> Laser Arcade Target Jumper

Commit message: Complete Target Jumper PCB
Parts:
- added J19, J20: I2C, 0_AKeller_Footprints:1x6_100mil_Header, symbol 0_AKeller_Parts:Header_1x6
- J1, J10, J11, J12, J13, J14, J15, J16, J17, J18, J2, J3, J4, J5, J6, J7, J8, J9: footprint (none) -> 0_AKeller_Footprints:1x6_100mil_Header
Connections:
- net +5V: now also J19.1, J19.2, J20.1, J20.2
- net GND: now also J19.5, J19.6, J20.5, J20.6
- net SCL: now reaches J1.3, J10.3, J11.3, J12.3, J13.3, J14.3, J15.3, J16.3, J17.3, J18.3, J2.3, J3.3, J4.3, J5.3, J6.3, J7.3, J8.3, J9.3
- net SCL: now also J19.3, J20.3
- net SDA: now reaches J1.4, J10.4, J11.4, J12.4, J13.4, J14.4, J15.4, J16.4, J17.4, J18.4, J2.4, J3.4, J4.4, J5.4, J6.4, J7.4, J8.4, J9.4
- net SDA: now also J19.4, J20.4
