File: KiCad/Target_Slave/Target_Slave.kicad_sch (KiCad schematic)
At the start: 48 parts, among them J1 ICSP, J10 I2C, J2 LED, J3 I2C, J4 I2C, J5 SERVO1, J6 SERVO3, J7 SERVO2, J8 Stepper, J9 I2C, U1 PIC16F1788-IP, U2 TSSP4038

Commit message: Rev B Target Slave PCB design
Parts:
- removed TP13: SERVO1, 0_AKeller_Footprints:1x1_100mil_Header, symbol 0_AKeller_Parts:Test_Point
- removed TP14: SERVO3, 0_AKeller_Footprints:1x1_100mil_Header, symbol 0_AKeller_Parts:Test_Point
- removed TP16: SERVO2, 0_AKeller_Footprints:1x1_100mil_Header, symbol 0_AKeller_Parts:Test_Point
- removed TP3: RGB_OUT, 0_AKeller_Footprints:1x1_100mil_Header, symbol 0_AKeller_Parts:Test_Point
- removed TP6: DIR, 0_AKeller_Footprints:1x1_100mil_Header, symbol 0_AKeller_Parts:Test_Point
- removed TP7: CLK, 0_AKeller_Footprints:1x1_100mil_Header, symbol 0_AKeller_Parts:Test_Point
- D1: footprint 0_AKeller_Footprints:Diode_0805 -> Diode_SMD:D_0805_2012Metric_Pad1.15x1.40mm_HandSolder
- J10, J3, J4, J9: footprint (none) -> 0_AKeller_Footprints:1x6_100mil_Header
- J2: footprint (none) -> 0_AKeller_Footprints:1x3_100mil_Header_Locking
- J5, J6, J7, JP1: footprint (none) -> 0_AKeller_Footprints:1x3_100mil_Header
- J8: footprint (none) -> 0_AKeller_Footprints:1x4_100mil_Header
- R1, R2, R3, R4, R5: footprint (none) -> Resistor_SMD:R_0805_2012Metric_Pad1.20x1.40mm_HandSolder
- renumbered TP15 to TP10, TP4 to TP3, TP5 to TP4, TP8 to TP5, TP9 to TP6, TP10 to TP7, TP11 to TP8, TP12 to TP9
Connections:
- net SCL: now reaches J10.3, J3.3, J4.3, J9.3, TP7.1, U1.14 (RC3/SCK/SCL)
- net SDA: now reaches J10.4, J3.4, J4.4, J9.4, TP8.1, U1.15 (RC4/SDI/SDA)
- net MCLR: now reaches D1.1 (K), J1.1, TP1.1, U1.1 (RE3/~{MCLR}/Vpp)
