File: KiCad/Target_Master/Target_Master.kicad_sch (KiCad schematic)
At the start: 13 parts, among them J2 ICSP, J3 I2C, J4 I2C, J5 I2C, U1 PIC16F1788-IP

Commit message: Completed Target Master Rev. B PCB
Parts:
- removed C6: 220uF, Capacitor_THT:CP_Radial_D6.3mm_P2.50mm, symbol Device:C_Polarized_Small_US
- removed C7: 0.1uF, Capacitor_SMD:C_0805_2012Metric_Pad1.18x1.45mm_HandSolder, symbol Device:C_Small
- removed J3, J4, J5: I2C, 0_AKeller_Footprints:1x4_100mil_Header, symbol Libraries:Header_1x4
- added J3, J4, J5: I2C, 0_AKeller_Footprints:1x6_100mil_Header, symbol 0_AKeller_Parts:Header_1x6
- added TP1: SCL, 0_AKeller_Footprints:1x1_100mil_Header, symbol 0_AKeller_Parts:Test_Point
- added TP2: SDA, 0_AKeller_Footprints:1x1_100mil_Header, symbol 0_AKeller_Parts:Test_Point
- D2: footprint 0_AKeller_Footprints:Diode_0805 -> Diode_SMD:D_0805_2012Metric_Pad1.15x1.40mm_HandSolder
- renumbered C4 to C6, C5 to C7
Connections:
- net +5V: now also J3.1, J3.2, J4.1, J4.2, J5.1, J5.2
- net GND: now also C6.1, C7.2, J3.5, J3.6, J4.5, J4.6, J5.5, J5.6
- net SCL: now reaches R3.2, U1.14 (RC3/SCK/SCL)
- net SCL: now also J3.3, J4.3, J5.3, TP1.1
- net SDA: now reaches R4.2, U1.15 (RC4/SDI/SDA)
- net SDA: now also J3.4, J4.4, J5.4, TP2.1
Other:
- note added: "1 = +5V 2 = +5V 3 = SCL 4 = SDA 5 = GND 6 = GND"
- note removed: "RC3, Pin 2 = SCL RC4, Pin 3 = SDA"
- moved on the sheet: C6, C7, D2, J2, R2, R3, R4, U1
