File: KiCad/Target_Master/Target_Power.kicad_sch (KiCad schematic)
At the start: 6 parts, among them J1 +5V

Commit message: Completed Target Master Rev. B PCB
Parts:
- added C4: 220uF, Capacitor_THT:CP_Radial_D6.3mm_P2.50mm, symbol Device:C_Polarized_Small_US
- added C5: 0.1uF, Capacitor_SMD:C_0805_2012Metric_Pad1.18x1.45mm_HandSolder, symbol Device:C_Small
Connections:
- net +5V: now also C4.1, C5.1
- net GND: now also C4.2, C5.2
