File: KiCad/Target_Master/UART.kicad_sch (KiCad schematic)
At the start: 18 parts, among them J6 USB_B_Mini, U2 FT232RL

Commit message: Completed Target Master Rev. B PCB
Parts:
- removed L1: 2uH, Inductor_SMD:L_0805_2012Metric_Pad1.15x1.40mm_HandSolder, symbol Device:L
- renumbered J6 to J7, TP1 to TP3, TP2 to TP4, TP3 to TP5, TP4 to TP6
Changed lines of the file:
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@@
 (kicad_sch
-	(version 20231120)
+	(version 20250114)
 	(generator "eeschema")
-	(generator_version "8.0")
+	(generator_version "9.0")
 	(paper "A")
 	(title_block
 		(title "Laser Arcade Master")
-		(date "2025-04-17")
-		(rev "A")
+		(date "2025-11-17")
+		(rev "B")
 		(company "Idaho State University")
+		(comment 1 "Andrew Keller")
 	)
 	(junction
@@
 	)
 	(junction
-		(at 73.66 86.36)
-		(diameter 0)
-		(color 0 0 0 0)
-	)
-	(junction
 		(at 104.14 104.14)
 		(diameter 0)
 		(color 0 0 0 0)
 	)
-	(junction
-		(at 104.14 86.36)
-		(diameter 0)
-		(color 0 0 0 0)
-	)
 	(no_connect
 		(at 167.64 99.06)
@@
 	(wire
 		(pts
-			(xy 92.71 86.36) (xy 104.14 86.36)
-		)
-		(stroke
-			(width 0)
-			(type default)
-		)
-	)
-	(wire
-		(pts
 			(xy 179.07 99.06) (xy 179.07 100.33)
 		)
@@
 		(pts
 			(xy 190.5 111.76) (xy 167.64 111.76)
-		)
-		(stroke
-			(width 0)
-			(type default)
-		)
-	)
-	(wire
-		(pts
-			(xy 73.66 86.36) (xy 85.09 86.36)
 		)
 		(stroke
@@
 		(dnp no)
 		(fields_autoplaced yes)
-		(property "Reference" "#PWR015"
+		(property "Reference" "#PWR016"
 			(at 119.38 90.17 0)
 			(effects
@@
 			(project "Target"
 				(path "/b95a4fbb-e866-40f1-8b06-3d5c3eea26d9/7a25075f-ac68-4e20-a244-e2abb088b838"
-					(reference "#PWR015")
+					(reference "#PWR016")
 					(unit 1)
 				)
@@
 		(dnp no)
 		(fields_autoplaced yes)
-		(property "Reference" "#PWR017"
+		(property "Reference" "#PWR018"
 			(at 127 135.89 0)
 			(effects
@@
 			(project "Target"
 				(path "/b95a4fbb-e866-40f1-8b06-3d5c3eea26d9/7a25075f-ac68-4e20-a244-e2abb088b838"
-					(reference "#PWR017")
+					(reference "#PWR018")
 					(unit 1)
 				)
@@
 		(dnp no)
 		(fields_autoplaced yes)
-		(property "Reference" "TP1"
+		(property "Reference" "TP3"
 			(at 168.91 77.724 0)
 			(do_not_autoplace yes)
@@
 			(project ""
 				(path "/b95a4fbb-e866-40f1-8b06-3d5c3eea26d9/7a25075f-ac68-4e20-a244-e2abb088b838"
-					(reference "TP1")
+					(reference "TP3")
 					(unit 1)
 				)
@@
 		(dnp no)
 		(fields_autoplaced yes)
-		(property "Reference" "TP4"
+		(property "Reference" "TP6"
 			(at 81.28 80.264 0)
 			(do_not_autoplace yes)
@@
 			(project "Target"
 				(path "/b95a4fbb-e866-40f1-8b06-3d5c3eea26d9/7a25075f-ac68-4e20-a244-e2abb088b838"
-					(reference "TP4")
+					(reference "TP6")
 					(unit 1)
 				)
@@
 		(dnp no)
 		(fields_autoplaced yes)
-		(property "Reference" "#+5V010"
+		(property "Reference" "#+5V011"
 			(at 203.2 82.55 0)
 			(effects
@@
 			(project "Target"
 				(path "/b95a4fbb-e866-40f1-8b06-3d5c3eea26d9/7a25075f-ac68-4e20-a244-e2abb088b838"
-					(reference "#+5V010")
+					(reference "#+5V011")
 					(unit 1)
 				)
@@
 		(dnp no)
 		(fields_autoplaced yes)
-		(property "Reference" "TP3"
+		(property "Reference" "TP5"
 			(at 77.47 80.264 0)
 			(do_not_autoplace yes)
@@
 			(project ""
 				(path "/b95a4fbb-e866-40f1-8b06-3d5c3eea26d9/7a25075f-ac68-4e20-a244-e2abb088b838"
-					(reference "TP3")
+					(reference "TP5")
 					(unit 1)
 				)
@@
 		(dnp no)
 		(fields_autoplaced yes)
-		(property "Reference" "TP2"
+		(property "Reference" "TP4"
 			(at 173.99 77.724 0)
 			(do_not_autoplace yes)
@@
 			(project "Target"
 				(path "/b95a4fbb-e866-40f1-8b06-3d5c3eea26d9/7a25075f-ac68-4e20-a244-e2abb088b838"
-					(reference "TP2")
+					(reference "TP4")
 					(unit 1)
 				)
@@
 		(dnp no)
 		(fields_autoplaced yes)
-		(property "Reference" "#PWR016"
+		(property "Reference" "#PWR017"
 			(at 57.15 111.76 0)
 			(effects
@@
 			(project "Target"
 				(path "/b95a4fbb-e866-40f1-8b06-3d5c3eea26d9/7a25075f-ac68-4e20-a244-e2abb088b838"
-					(reference "#PWR016")
+					(reference "#PWR017")
 					(unit 1)
 				)
@@
 		(dnp no)
 		(fields_autoplaced yes)
-		(property "Reference" "#+5V09"
+		(property "Reference" "#+5V010"
 			(at 149.86 68.58 0)
 			(effects
@@
 			(project "Target"
 				(path "/b95a4fbb-e866-40f1-8b06-3d5c3eea26d9/7a25075f-ac68-4e20-a244-e2abb088b838"
-					(reference "#+5V09")
+					(reference "#+5V010")
 					(unit 1)
 				)
@@
 	)
 	(symbol
-		(lib_id "Device:L")
-		(at 88.9 86.36 90)
-		(unit 1)
-		(exclude_from_sim no)
-		(in_bom yes)
-		(on_board yes)
-		(dnp no)
-		(fields_autoplaced yes)
-		(property "Reference" "L1"
-			(at 88.9 81.28 90)
-			(effects
-				(font
-					(size 1.27 1.27)
-				)
-			)
-		)
-		(property "Value" "2uH"
-			(at 88.9 83.82 90)
-			(effects
-				(font
-					(size 1.27 1.27)
-				)
-			)
-		)
-		(property "Footprint" "Inductor_SMD:L_0805_2012Metric_Pad1.15x1.40mm_HandSolder"
-			(at 88.9 86.36 0)
-			(effects
-				(font
-					(size 1.27 1.27)
-				)
-				(hide yes)
-			)
-		)
-		(property "Datasheet" "~"
-			(at 88.9 86.36 0)
-			(effects
-				(font
-					(size 1.27 1.27)
-				)
-				(hide yes)
-			)
-		)
-		(property "Description" "Inductor"
-			(at 88.9 86.36 0)
-			(effects
-				(font
-					(size 1.27 1.27)
-				)
-				(hide yes)
-			)
-		)
-		(pin "1"
-		)
-		(pin "2"
-		)
-		(instances
-			(project "Target"
-				(path "/b95a4fbb-e866-40f1-8b06-3d5c3eea26d9/7a25075f-ac68-4e20-a244-e2abb088b838"
-					(reference "L1")
-					(unit 1)
-				)
-			)
-		)
-	)
-	(symbol
 		(lib_id "Libraries:R_Custom")
 		(at 179.07 104.14 90)
@@
 		(dnp no)
 		(fields_autoplaced yes)
-		(property "Reference" "J6"
+		(property "Reference" "J7"
 			(at 59.69 78.74 0)
 			(effects
@@
 			(project "Target"
 				(path "/b95a4fbb-e866-40f1-8b06-3d5c3eea26d9/7a25075f-ac68-4e20-a244-e2abb088b838"
-					(reference "J6")
+					(reference "J7")
 					(unit 1)
 				)
