File: KiCad/Target_Master/Target.kicad_pcb (KiCad board)
At the start: 2 copper layers, 76.2 x 50.8 mm, 45 parts, among them J1 +5V, J2 ICSP, J3 I2C, J4 I2C, J5 I2C, J6 USB_B_Mini, U1 PIC16F1788-IP, U2 FT232RL

Commit message: Completed Target Master Rev. B PCB
Parts:
- removed the G*** at (124.5, 108.7)
- removed the G*** at (130.2, 109.3)
- removed J6: USB_B_Mini, 0_AKeller_Footprints:USB_Micro-B_Amphenol
- removed L1: 2uH, Inductor_SMD:L_0805_2012Metric_Pad1.15x1.40mm_HandSolder
- added G***: LOGO, 2025 Logos:RCET Horizontal 23x155, F.Cu at (173.4, 103.0)
- added G***: LOGO, 2025 Logos:LA_QR_Code_0-5x0-5, B.Cu at (132.8, 110.9)
- added J7: USB_B_Mini, 0_AKeller_Footprints:USB_Micro-B_Amphenol, F.Cu at (113.7, 108.2)
- added TP5: ~, 0_AKeller_Footprints:1x1_100mil_Header, F.Cu at (123.2, 110.0)
- added TP6: ~, 0_AKeller_Footprints:1x1_100mil_Header, F.Cu at (123.2, 107.2)
- C10, C11, C12, C13, C3, R1, R2, R3, R4: moved to F.Cu
- C4: value 1uF -> 220uF; footprint Capacitor_SMD:C_0805_2012Metric_Pad1.18x1.45mm_HandSolder -> Capacitor_THT:CP_Radial_D6.3mm_P2.50mm; moved to F.Cu
- C5: value 1uF -> 0.1uF; moved to F.Cu
- C6: value 220uF -> 1uF; footprint Capacitor_THT:CP_Radial_D6.3mm_P2.50mm -> Capacitor_SMD:C_0805_2012Metric_Pad1.18x1.45mm_HandSolder
- C7: value 0.1uF -> 1uF
- D2: footprint 0_AKeller_Footprints:Diode_0805 -> Diode_SMD:D_0805_2012Metric_Pad1.15x1.40mm_HandSolder; moved to F.Cu
- J3, J4, J5: footprint 0_AKeller_Footprints:1x4_100mil_Header -> 0_AKeller_Footprints:1x6_100mil_Header
- TP1: value ~ -> SCL
- TP2: value ~ -> SDA
- moved G*** 55.4 mm to (168.8, 84.3)
- moved C5 45.5 mm to (123.8, 79.0), turned to 180 degrees
- moved R4 41.1 mm to (163.4, 76.5), turned to 90 degrees
- moved R3 36.8 mm to (167.5, 76.5), turned to 90 degrees
- moved J4 36.3 mm to (148.6, 120.1)
- moved C4 34.8 mm to (129.6, 79.8), turned to 0 degrees
- moved J3 31.4 mm to (148.6, 77.0)
- moved C13 30.9 mm to (133.2, 121.4), turned to -90 degrees
- moved C12 30.9 mm to (129.5, 121.4), turned to -90 degrees
- moved C6 30.5 mm to (153.0, 108.2), turned to -90 degrees
- moved J1 27.7 mm to (123.5, 88.9), turned to 90 degrees
- moved J2 26.2 mm to (167.9, 98.6), turned to -90 degrees
- moved C7 24.4 mm to (150.6, 86.7), turned to 180 degrees
- moved TP2 24.1 mm to (159.8, 85.2)
- moved D1 22.1 mm to (134.1, 98.8), turned to 180 degrees
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Connections:
- C10 pad 1: Net-(J6-D-) -> Net-(J7-D-)
- C11 pad 1: Net-(J6-D+) -> Net-(J7-D+)
- C4 pad 1: GND -> +5V
- C4 pad 2: +5V -> GND
- C5 pad 1: Net-(D2-A) -> +5V
- C6 pad 1: +5V -> GND
- C6 pad 2: GND -> +5V
- C7 pad 1: +5V -> Net-(D2-A)
- J3 pad 2: Net-(U1-RC3/SCK/SCL) -> +5V
- J3 pad 3: Net-(U1-RC4/SDI/SDA) -> /Master/SCL
- J3 pad 4: GND -> /Master/SDA
- J4 pad 2: Net-(U1-RC3/SCK/SCL) -> +5V
- J4 pad 3: Net-(U1-RC4/SDI/SDA) -> /Master/SCL
- J4 pad 4: GND -> /Master/SDA
- J5 pad 2: Net-(U1-RC3/SCK/SCL) -> +5V
- J5 pad 3: Net-(U1-RC4/SDI/SDA) -> /Master/SCL
- J5 pad 4: GND -> /Master/SDA
- R3 pad 2: Net-(U1-RC3/SCK/SCL) -> /Master/SCL
- R4 pad 2: Net-(U1-RC4/SDI/SDA) -> /Master/SDA
- TP1 pad 1: RX -> /Master/SCL
- TP2 pad 1: TX -> /Master/SDA
- TP3 pad 1: Net-(J6-D+) -> RX
- TP4 pad 1: Net-(J6-D-) -> TX
- U1 pad 14: Net-(U1-RC3/SCK/SCL) -> /Master/SCL
- U1 pad 15: Net-(U1-RC4/SDI/SDA) -> /Master/SDA
- U2 pad 15: Net-(J6-D+) -> Net-(J7-D+)
- U2 pad 16: Net-(J6-D-) -> Net-(J7-D-)
Routing:
- net /Master/SDA: track 0.00 -> 152.2 mm
- net /Master/SCL: track 0.00 -> 141.1 mm
- net Net-(U1-RC4/SDI/SDA): track 61.7 -> 0.00 mm
- net Net-(U1-RC3/SCK/SCL): track 49.0 -> 0.00 mm
- net Net-(J6-D-): track 34.5 -> 0.00 mm
- net Net-(J6-D+): track 33.5 -> 0.00 mm
- net GND: track 43.0 -> 67.5 mm, vias 3 -> 0
- net Net-(J7-D-): track 0.00 -> 23.9 mm
- net Net-(J7-D+): track 0.00 -> 17.1 mm
- net +5V: track 232.9 -> 239.8 mm
- net TX: track 31.4 -> 25.3 mm
- net Net-(J7-VBUS): track 12.1 -> 6.69 mm
- net Net-(D2-K): track 21.3 -> 16.3 mm
- net RB6: track 18.2 -> 13.3 mm
- net RB7: track 16.4 -> 11.5 mm
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Other:
- board text added: "Laser Arcade Target Master Rev. B - Fall 2025"
- board text removed: "I2C"
- board text removed: "ICSP"
- board text removed: "Laser Arcade Target Master Rev. A Spring 2025"
- board text removed: "PWR"
- board text removed: "RX"
- board text removed: "TX"

Commit message: Completed Target Master PCB, export gerbers and views
Parts:
- J7: value USB_B_Mini -> USB_B_Micro
